Commit message: [fix] Bundle UR5 meshes to make combined robot assets portable

File: assets/ur5_inspire/robot_ur5_inspire.urdf (robot description, URDF)
Before this commit: robot ur5_inspire, 19 links, 18 joints
Links:
- link base_link: geometry collision mesh filename=meshes_ur5_inspire/ur5_base_ur5_inspire.stl; visual mesh filename=meshes_ur5_inspire/ur5_base_ur5_inspire.stl
- link forearm_link: geometry collision mesh filename=meshes_ur5_inspire/ur5_forearm_ur5_inspire.stl; visual mesh filename=meshes_ur5_inspire/ur5_forearm_ur5_inspire.stl
- link shoulder_link: geometry collision mesh filename=meshes_ur5_inspire/ur5_shoulder_ur5_inspire.stl; visual mesh filename=meshes_ur5_inspire/ur5_shoulder_ur5_inspire.stl
- link upper_arm_link: geometry collision mesh filename=meshes_ur5_inspire/ur5_upperarm_ur5_inspire.stl; visual mesh filename=meshes_ur5_inspire/ur5_upperarm_ur5_inspire.stl
- link wrist_1_link: geometry collision mesh filename=meshes_ur5_inspire/ur5_wrist1_ur5_inspire.stl; visual mesh filename=meshes_ur5_inspire/ur5_wrist1_ur5_inspire.stl
- link wrist_2_link: geometry collision mesh filename=meshes_ur5_inspire/ur5_wrist2_ur5_inspire.stl; visual mesh filename=meshes_ur5_inspire/ur5_wrist2_ur5_inspire.stl
- link wrist_3_link: geometry collision mesh filename=meshes_ur5_inspire/ur5_wrist3_ur5_inspire.stl; visual mesh filename=meshes_ur5_inspire/ur5_wrist3_ur5_inspire.stl
